File: fauxmac-plus.kicad_pcb (KiCad board)
At the start: 2 copper layers, 86.5 x 89 mm, 42 parts, among them U1 

Commit message: 2023 updates to PCB with RGB and plates
Parts:
- removed  : oled, keyboardio:4P-2.0-no-outline
- added J1: oled, Connector_PinHeader_2.54mm:PinHeader_1x04_P2.54mm_Vertical, F.Cu at (141.3, 64.0)
- added dout: TestPoint, Connector_PinSocket_2.54mm:PinSocket_1x01_P2.54mm_Vertical, F.Cu at (137.5, 111.6)
- added gnd: TestPoint, Connector_PinSocket_2.54mm:PinSocket_1x01_P2.54mm_Vertical, F.Cu at (142.1, 111.6)
- added rgb1: WS2812B, LED_SMD:LED_WS2812B_PLCC4_5.0x5.0mm_P3.2mm, B.Cu at (135.8, 36.6)
- added rgb2: WS2812B, LED_SMD:LED_WS2812B_PLCC4_5.0x5.0mm_P3.2mm, B.Cu at (188.7, 34.4)
- added rgb3: WS2812B, LED_SMD:LED_WS2812B_PLCC4_5.0x5.0mm_P3.2mm, B.Cu at (188.1, 107.6)
- added rgb4: WS2812B, LED_SMD:LED_WS2812B_PLCC4_5.0x5.0mm_P3.2mm, B.Cu at (137.5, 107.9)
- added vcc: TestPoint, Connector_PinSocket_2.54mm:PinSocket_1x01_P2.54mm_Vertical, F.Cu at (132.9, 111.6)
- H1, H2, H3, H4, K10, K11, K12, K2, K3, K4, K5, K6, K7, K8, K9, on/off: renamed from  
- K1: renamed from   
- U1: value (none) -> ProMicro
- moved col1 2.50 mm to (137.5, 104.0)
- renumbered POS to batt+, NEG to batt-
Connections:
- U1 pad 12: Net-(U1-Pad12) -> rgb
- U1 pad 21: Net-(U1-Pad21) -> unconnected-(U1-Pad21)
- U1 pad 22: Net-(U1-Pad22) -> unconnected-(U1-Pad22)
- U1 pad 23: Net-(U1-Pad23) -> unconnected-(U1-Pad23)
- U1 pad 24: Net-(U1-Pad24) -> unconnected-(U1-Pad24)
- U1 pad 8: Net-(U1-Pad8) -> unconnected-(U1-Pad8)
- U1 pad 9: Net-(U1-Pad9) -> unconnected-(U1-Pad9)
Routing:
- net VCC: track 35.0 -> 199.2 mm, vias 1 -> 4
- net Net-(rgb2-Pad2): track 0.00 -> 104.2 mm
- net GND: track 211.4 -> 295.2 mm, vias 1 -> 3
- net Net-(rgb1-Pad2): track 0.00 -> 62.0 mm, vias 0 -> 2
- net Net-(rgb3-Pad2): track 0.00 -> 47.4 mm, vias 0 -> 2
- net rgb: track 0.00 -> 30.4 mm, vias 0 -> 2
- net Net-(rgb4-Pad2): track 0.00 -> 9.52 mm, vias 0 -> 2
- net col1: track 150.9 -> 148.4 mm
- net sda: track 24.0 -> 23.4 mm
- added copper zone on B.Cu, net (none)
- added copper zone on F.Cu, net (none)
Other:
- net class Default removed
- board text added: "The controller goes on this side, chip facing upwards/outwards"
